File: electronics/bluetooth_shield/bluetooth_shield.sch (KiCad schematic (older format))
At the start: 6 parts, among them IC1 453-00005, J1 Conn_02x08_Odd_Even, J2 Conn_01x03_Male, J3 Conn_01x04_Male, U1 AP2127R-3.3

Commit message: Updating layouts and schematics and reading for export
Parts:
- removed J2: Conn_01x03_Male, Connector_PinHeader_2.54mm:PinHeader_1x03_P2.54mm_Vertical, symbol Connector:Conn_01x03_Male
- removed J3: Conn_01x04_Male, Connector_PinHeader_2.54mm:PinHeader_1x04_P2.54mm_Vertical, symbol Connector:Conn_01x04_Male
- added H1, H2: MountingHole, MountingHole:MountingHole_3.2mm_M3_DIN965_Pad_TopBottom, symbol Mechanical:MountingHole
- added J2, J3: Conn_01x05_Male, Connector_PinHeader_2.54mm:PinHeader_1x05_P2.54mm_Vertical, symbol Connector:Conn_01x05_Male
- C1: footprint (none) -> Capacitor_SMD:C_0805_2012Metric_Pad1.18x1.45mm_HandSolder
Connections:
- net GND: now also J2.5 (Pin_5), J3.1 (Pin_1)
- net at IC1.17 (P0.08/UART_RX): now also J2.1 (Pin_1)
- net at IC1.18 (P0.07/UART_CTS): now also J2.2 (Pin_2)
- net at IC1.19 (P0.06/UART_TX): now also J2.3 (Pin_3)
- net at IC1.20 (P0.05/UART_RTS/_AIN3): now also J2.4 (Pin_4)
- net VDD: now reaches C1.1, IC1.26 (VDD_NRF), U1.3 (VO)
- net VDD: now also J3.5 (Pin_5)
- net at IC1.5 (SWDIO): now also J3.2 (Pin_2)
- net at IC1.6 (SWDCLK): now also J3.3 (Pin_3)
- net at IC1.7 (NRESET/_P0.21): now also J3.4 (Pin_4)
Changed lines of the file:
@@
 	7500 1150 8200 1150
 Wire Wire Line
-	8200 1150 8200 1300
+	8200 1150 8200 1200
 $Comp
 L power:GND #PWR0104
 U 1 1 615111CD
-P 8200 1300
-F 0 "#PWR0104" H 8200 1050 50  0001 C CNN
-F 1 "GND" H 8205 1127 50  0000 C CNN
-F 2 "" H 8200 1300 50  0001 C CNN
-F 3 "" H 8200 1300 50  0001 C CNN
-	1    8200 1300
-	1    0    0    -1
-$EndComp
-Wire Wire Line
-	7500 2650 8200 2650
+P 8200 1200
+F 0 "#PWR0104" H 8200 950 50  0001 C CNN
+F 1 "GND" H 8205 1027 50  0000 C CNN
+F 2 "" H 8200 1200 50  0001 C CNN
+F 3 "" H 8200 1200 50  0001 C CNN
+	1    8200 1200
+	1    0    0    -1
+$EndComp
 Wire Wire Line
 	8200 2650 8200 2800
@@
 $EndComp
 Wire Wire Line
-	5100 1750 4400 1750
-Wire Wire Line
-	4400 1750 4400 1900
+	5100 1750 4550 1750
+Wire Wire Line
+	4550 1750 4550 1900
 $Comp
 L power:GND #PWR0107
 U 1 1 6151352B
-P 4400 1900
-F 0 "#PWR0107" H 4400 1650 50  0001 C CNN
-F 1 "GND" H 4405 1727 50  0000 C CNN
-F 2 "" H 4400 1900 50  0001 C CNN
-F 3 "" H 4400 1900 50  0001 C CNN
-	1    4400 1900
+P 4550 1900
+F 0 "#PWR0107" H 4550 1650 50  0001 C CNN
+F 1 "GND" H 4555 1727 50  0000 C CNN
+F 2 "" H 4550 1900 50  0001 C CNN
+F 3 "" H 4550 1900 50  0001 C CNN
+	1    4550 1900
 	-1   0    0    -1
 $EndComp
@@
 F 0 "C1" H 4265 1946 50  0000 L CNN
 F 1 "C" H 4265 1855 50  0000 L CNN
-F 2 "" H 4188 1750 50  0001 C CNN
+F 2 "Capacitor_SMD:C_0805_2012Metric_Pad1.18x1.45mm_HandSolder" H 4188 1750 50  0001 C CNN
 F 3 "~" H 4150 1900 50  0001 C CNN
 	1    4150 1900
@@
 Connection ~ 4150 1650
 Wire Wire Line
-	4150 1650 5100 1650
+	4150 1650 4550 1650
 $Comp
 L power:GND #PWR0108
@@
 	1    0    0    -1
 $EndComp
-$Comp
-L Connector:Conn_01x03_Male J2
-U 1 1 6151C72C
-P 8000 1650
-F 0 "J2" H 7972 1674 50  0000 R CNN
-F 1 "Conn_01x03_Male" H 7972 1583 50  0000 R CNN
-F 2 "Connector_PinHeader_2.54mm:PinHeader_1x03_P2.54mm_Vertical" H 8000 1650 50  0001 C CNN
-F 3 "~" H 8000 1650 50  0001 C CNN
-	1    8000 1650
-	-1   0    0    -1
-$EndComp
-Wire Wire Line
-	7800 1550 7500 1550
-Wire Wire Line
-	7800 1650 7500 1650
-Wire Wire Line
-	7500 1750 7800 1750
-$Comp
-L Connector:Conn_01x04_Male J3
-U 1 1 61521B68
-P 8000 2850
-F 0 "J3" H 7972 2824 50  0000 R CNN
-F 1 "Conn_01x04_Male" H 7972 2733 50  0000 R CNN
-F 2 "Connector_PinHeader_2.54mm:PinHeader_1x04_P2.54mm_Vertical" H 8000 2850 50  0001 C CNN
-F 3 "~" H 8000 2850 50  0001 C CNN
-	1    8000 2850
-	-1   0    0    -1
-$EndComp
+Wire Wire Line
+	8700 1550 7500 1550
+Wire Wire Line
+	8700 1650 7500 1650
+Wire Wire Line
+	7500 1750 8700 1750
 Wire Wire Line
 	7800 2750 7500 2750
@@
 Wire Wire Line
 	4150 1750 4150 1650
+$Comp
+L power:GND #PWR04
+U 1 1 61532346
+P 8600 1950
+F 0 "#PWR04" H 8600 1700 50  0001 C CNN
+F 1 "GND" H 8605 1777 50  0000 C CNN
+F 2 "" H 8600 1950 50  0001 C CNN
+F 3 "" H 8600 1950 50  0001 C CNN
+	1    8600 1950
+	1    0    0    -1
+$EndComp
+$Comp
+L power:VDD #PWR01
+U 1 1 615339A1
+P 4550 1450
+F 0 "#PWR01" H 4550 1300 50  0001 C CNN
+F 1 "VDD" H 4565 1623 50  0000 C CNN
+F 2 "" H 4550 1450 50  0001 C CNN
+F 3 "" H 4550 1450 50  0001 C CNN
+	1    4550 1450
+	1    0    0    -1
+$EndComp
+Wire Wire Line
+	4550 1450 4550 1650
+Connection ~ 4550 1650
+Wire Wire Line
+	4550 1650 5100 1650
+$Comp
+L power:VDD #PWR03
+U 1 1 61534F48
+P 8550 1300
+F 0 "#PWR03" H 8550 1150 50  0001 C CNN
+F 1 "VDD" H 8565 1473 50  0000 C CNN
+F 2 "" H 8550 1300 50  0001 C CNN
+F 3 "" H 8550 1300 50  0001 C CNN
+	1    8550 1300
+	1    0    0    -1
+$EndComp
+Wire Wire Line
+	7500 2650 8200 2650
+$Comp
+L Connector:Conn_01x05_Male J2
+U 1 1 61543302
+P 8000 2950
+F 0 "J2" H 7972 2924 50  0000 R CNN
+F 1 "Conn_01x05_Male" H 7972 2833 50  0001 R CNN
+F 2 "Connector_PinHeader_2.54mm:PinHeader_1x05_P2.54mm_Vertical" H 8000 2950 50  0001 C CNN
+F 3 "~" H 8000 2950 50  0001 C CNN
+	1    8000 2950
+	-1   0    0    -1
+$EndComp
+$Comp
+L power:GND #PWR02
+U 1 1 615443E6
+P 7650 3250
+F 0 "#PWR02" H 7650 3000 50  0001 C CNN
+F 1 "GND" H 7655 3077 50  0000 C CNN
+F 2 "" H 7650 3250 50  0001 C CNN
+F 3 "" H 7650 3250 50  0001 C CNN
+	1    7650 3250
+	1    0    0    -1
+$EndComp
+Wire Wire Line
+	7650 3250 7650 3150
+Wire Wire Line
+	7650 3150 7800 3150
+$Comp
+L Connector:Conn_01x05_Male J3
+U 1 1 61531D5C
+P 8900 1650
+F 0 "J3" H 8872 1624 50  0000 R CNN
+F 1 "Conn_01x05_Male" H 8872 1533 50  0001 R CNN
+F 2 "Connector_PinHeader_2.54mm:PinHeader_1x05_P2.54mm_Vertical" H 8900 1650 50  0001 C CNN
+F 3 "~" H 8900 1650 50  0001 C CNN
+	1    8900 1650
+	-1   0    0    -1
+$EndComp
+Wire Wire Line
+	8550 1850 8700 1850
+Wire Wire Line
+	8550 1300 8550 1850
+Wire Wire Line
+	8600 1950 8600 1450
+Wire Wire Line
+	8600 1450 8700 1450
+$Comp
+L Mechanical:MountingHole H1
+U 1 1 61566D42
+P 3400 4400
+F 0 "H1" H 3500 4446 50  0000 L CNN
+F 1 "MountingHole" H 3500 4355 50  0000 L CNN
+F 2 "MountingHole:MountingHole_3.2mm_M3_DIN965_Pad_TopBottom" H 3400 4400 50  0001 C CNN
+F 3 "~" H 3400 4400 50  0001 C CNN
+	1    3400 4400
+	1    0    0    -1
+$EndComp
+$Comp
+L Mechanical:MountingHole H2
+U 1 1 61566DE7
+P 3400 4600
+F 0 "H2" H 3500 4646 50  0000 L CNN
+F 1 "MountingHole" H 3500 4555 50  0000 L CNN
+F 2 "MountingHole:MountingHole_3.2mm_M3_DIN965_Pad_TopBottom" H 3400 4600 50  0001 C CNN
+F 3 "~" H 3400 4600 50  0001 C CNN
+	1    3400 4600
+	1    0    0    -1
+$EndComp
 $EndSCHEMATC
